File: Work Bench 3.0.kicad_pcb (KiCad board)
At the start: 2 copper layers, 136 parts, among them J1 GND(A), J10 Lights 1 GND, J11 USB_A_Stacked, J12 Lights 2 GND, J13 Conn_01x02_Pin, J14 Lights 5V+(B), J15 Lights 1 GND, J16 Lights +5V(B), J17 Controls, J18 Lights 3 GND, J19 USB_A_Stacked, J2 GND(B), J20 Lights 4 GND, J21 Lights 4 GND, J22 Display, J23 Lights +5V(c), J24 Lights +5V(C), J25 Lights 3 GND, J26 Lights 5 GND, J27 Screw_Terminal_01x04, J28 Lights 6 GND, J29 Controls, J3 GND(C), J30 Lights 6 GND, J31 Lights +12V, J32 Lights +12V, J33 Lights 5 GND, J34 Extractor 1, J35 Extractor 2, J36 Extractor 3, J4 GND(12V), J5 +5V(A), J6 +5V(B), J7 +5V(C), J8 +12V, J9 Lights 2 GND, Q1 PMV20XNEAR, Q2 PMV20XNEAR, Q3 PMV20XNEAR, Q4 PMV20XNEAR, Q5 PMV20XNEAR, Q6 PMV20XNEAR, Q7 PMV20XNER, Q8 A2SHB, SW1 FSM4JSMA, SW2 FSM4JSMA, SW3 RotaryEncoder_Switch, U1 BCP5610TA, U10 BCP5610TA, U11 BCP53TA, U12 BCP5610TA, U13 BCP53TA, U2 BCP53TA, U3 Pico, U4 BCP5610TA, U5 BCP53TA, U6 BCP5610TA, U7 BCP53TA, U8 BCP5610TA, U9 BCP53TA

Commit message: Done
Parts:
- removed J15: Lights 1 GND, Connector_Wire:SolderWirePad_1x01_SMD_5x10mm
- removed J16: Lights +5V(B), Connector_Wire:SolderWirePad_1x01_SMD_5x10mm
- removed J18, J25: Lights 3 GND, Connector_Wire:SolderWirePad_1x01_SMD_5x10mm
- removed J20, J21: Lights 4 GND, Connector_Wire:SolderWirePad_1x01_SMD_5x10mm
- removed J23: Lights +5V(c), Connector_Wire:SolderWirePad_1x01_SMD_5x10mm
- removed J24: Lights +5V(C), Connector_Wire:SolderWirePad_1x01_SMD_5x10mm
- removed J26, J33: Lights 5 GND, Connector_Wire:SolderWirePad_1x01_SMD_5x10mm
- removed J28, J30: Lights 6 GND, Connector_Wire:SolderWirePad_1x01_SMD_5x10mm
- removed J31, J32: Lights +12V, Connector_Wire:SolderWirePad_1x01_SMD_5x10mm
- added J37: Conn_01x04_Pin, SMD-Connectors:SMD-PinHeader_1x04_P2.54mm_Vertical, F.Cu at (84.3, 35.8)
- added J38: 5V Lights, SMD-Connectors:SMD-PinHeader_1x04_P2.54mm_Vertical, F.Cu at (183.2, 60.5)
- J10: value Lights 1 GND -> Conn_01x02_Pin; footprint Connector_Wire:SolderWirePad_1x01_SMD_5x10mm -> SMD-Connectors:SMD-PinHeader_1x02_P2.54mm_Vertical
- J12: value Lights 2 GND -> GND(12V)
- J14: value Lights 5V+(B) -> +12V
- J9: value Lights 2 GND -> Conn_01x02_Pin; footprint Connector_Wire:SolderWirePad_1x01_SMD_5x10mm -> SMD-Connectors:SMD-PinHeader_1x02_P2.54mm_Vertical
- moved J14 216.4 mm to (243.8, 40.2)
- moved J12 206.4 mm to (236.2, 40.2)
- moved J10 150.0 mm to (183.2, 83.3)
- moved J9 97.6 mm to (132.8, 36.7), turned to 180 degrees
- moved C31 96.5 mm to (110.8, 180.1)
- moved J29 96.5 mm to (71.1, 138.4)
- moved R21 96.5 mm to (110.8, 142.1)
- moved R24 96.5 mm to (102.6, 184.5)
- moved SW1 96.5 mm to (56.0, 159.7)
- moved SW2 96.5 mm to (56.0, 167.3)
- moved SW3 96.5 mm to (104.2, 170.7)
- moved C18 96.5 mm to (49.8, 152.2)
- moved C23 96.5 mm to (49.8, 174.8)
- moved C28 96.5 mm to (102.6, 180.1)
- moved C29 96.5 mm to (110.8, 146.1)
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Connections:
- C13 pad 1: Net-(J19-VBUS1) -> +5V(C)
- C13 pad 2: Net-(J18-Pin_1) -> Net-(J19-GND1)
- C14 pad 1: Net-(J19-VBUS1) -> +5V(C)
- C22 pad 1: Net-(J27-Pin_2) -> +12V
- C22 pad 2: Net-(J26-Pin_1) -> Net-(J27-Pin_1)
- C24 pad 1: Net-(J27-Pin_2) -> +12V
- C6 pad 1: Net-(J11-VBUS1) -> +5V(B)
- C6 pad 2: Net-(J10-Pin_1) -> Net-(J11-GND1)
- C8 pad 1: Net-(J11-VBUS1) -> +5V(B)
- J11 pad 1: Net-(J11-VBUS1) -> +5V(B)
- J11 pad 4: Net-(J10-Pin_1) -> Net-(J11-GND1)
- J11 pad 5: Net-(J11-VBUS1) -> +5V(B)
- J12 pad 1: Net-(J11-GND2) -> GND
- J14 pad 1: +5V(B) -> +12V
- J19 pad 1: Net-(J19-VBUS1) -> +5V(C)
- J19 pad 4: Net-(J18-Pin_1) -> Net-(J19-GND1)
- J19 pad 5: Net-(J19-VBUS1) -> +5V(C)
- J27 pad 1: Net-(J26-Pin_1) -> Net-(J27-Pin_1)
- J27 pad 2: Net-(J27-Pin_2) -> +12V
- J27 pad 4: Net-(J27-Pin_2) -> +12V
- Q1 pad 3: Net-(J9-Pin_1) -> Net-(J11-GND2)
- Q2 pad 3: Net-(J15-Pin_1) -> Net-(J11-GND1)
- Q3 pad 3: Net-(J21-Pin_1) -> Net-(J19-GND2)
- Q4 pad 3: Net-(J25-Pin_1) -> Net-(J19-GND1)
- Q5 pad 3: Net-(J30-Pin_1) -> Net-(J27-Pin_3)
- Q6 pad 3: Net-(J33-Pin_1) -> Net-(J27-Pin_1)
- R10 pad 1: /Lights 4 Signal -> Net-(J37-Pin_4)
- R15 pad 1: /Lights 3 Signal -> Net-(J37-Pin_3)
- R2 pad 1: /Lights 2 Signal -> Net-(J37-Pin_2)
- R20 pad 1: /Lights 6 Signal -> Net-(J9-Pin_2)
- R26 pad 1: /Lights 5 Signal -> Net-(J9-Pin_1)
- R6 pad 1: /Lights 1 Signal -> Net-(J37-Pin_1)
- U3 pad 11: /Lights 4 Signal -> Net-(J38-Pin_4)
- U3 pad 14: /Lights 5 Signal -> Net-(J10-Pin_1)
- U3 pad 16: /Lights 6 Signal -> Net-(J10-Pin_2)
- U3 pad 4: /Lights 1 Signal -> Net-(J38-Pin_1)
- U3 pad 6: /Lights 2 Signal -> Net-(J38-Pin_2)
- U3 pad 9: /Lights 3 Signal -> Net-(J38-Pin_3)
Routing:
- net /Lights 1 Signal: track 133.1 -> 0.00 mm
- net /Lights 2 Signal: track 125.5 -> 0.00 mm
- net /Lights 3 Signal: track 106.1 -> 0.00 mm
- net /Lights 4 Signal: track 98.5 -> 0.00 mm
- net Net-(D1-A): track 115.8 -> 192.9 mm
- net Net-(J27-Pin_2): track 72.0 -> 0.00 mm
- net Net-(J37-Pin_2): track 0.00 -> 63.6 mm
- net /Lights 5 Signal: track 61.1 -> 0.00 mm
- net Net-(J37-Pin_1): track 0.00 -> 59.7 mm
- net /Lights 6 Signal: track 52.2 -> 0.00 mm
- net Net-(J18-Pin_1): track 43.9 -> 0.00 mm
- net +12V: track 359.7 -> 318.0 mm
- net Net-(J26-Pin_1): track 41.0 -> 0.00 mm
- net Net-(J11-GND1): track 0.00 -> 36.8 mm
- net Net-(J19-GND1): track 0.00 -> 36.7 mm
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- added copper zone on F.Cu, net Net-(J11-GND1)
- added copper zone on F.Cu, net Net-(J11-GND2)
- added copper zone on F.Cu, net Net-(J19-GND1)
- added copper zone on F.Cu, net Net-(J19-GND2)
- added copper zone on F.Cu, net Net-(J27-Pin_1)
- added copper zone on F.Cu, net Net-(J27-Pin_3)
- removed copper zone on F.Cu, net Net-(J15-Pin_1)
- removed copper zone on F.Cu, net Net-(J21-Pin_1)
- removed copper zone on F.Cu, net Net-(J25-Pin_1)
- removed copper zone on F.Cu, net Net-(J30-Pin_1)
- removed copper zone on F.Cu, net Net-(J33-Pin_1)
- removed copper zone on F.Cu, net Net-(J9-Pin_1)

Commit message: Split
Parts:
- removed J37: Conn_01x04_Pin, SMD-Connectors:SMD-PinHeader_1x04_P2.54mm_Vertical
- added J15: Conn_01x02_Pin, SMD-Connectors:SMD-PinHeader_1x02_P2.54mm_Vertical, F.Cu at (106.7, 121.8)
- added J16: Conn_01x02_Pin, SMD-Connectors:SMD-PinHeader_1x02_P2.54mm_Vertical, F.Cu at (63.8, 121.9)
- moved C18 153.4 mm to (199.7, 119.5)
- moved SW1 153.4 mm to (205.8, 127.0)
- moved R13 153.1 mm to (199.7, 114.8)
- moved C23 152.7 mm to (199.7, 145.6)
- moved C28 152.7 mm to (252.5, 150.9)
- moved R18 152.7 mm to (199.7, 150.5)
- moved R24 152.7 mm to (252.5, 155.3)
- moved C31 152.7 mm to (260.7, 150.9)
- moved J29 152.7 mm to (221.0, 109.2)
- moved R21 152.7 mm to (260.7, 112.9)
- moved SW2 152.7 mm to (205.8, 138.1)
- moved SW3 152.7 mm to (254.0, 141.5)
- moved C29 152.7 mm to (260.7, 116.8)
- moved R29 152.7 mm to (260.6, 155.3)
- moved J13 94.7 mm to (89.6, 36.0)
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Routing:
- net Net-(J16-Pin_2): track 63.6 -> 11.5 mm
- net Net-(J16-Pin_1): track 59.7 -> 20.2 mm
- net Net-(J13-Pin_2): track 0.00 -> 11.7 mm
- net Net-(J13-Pin_1): track 0.00 -> 11.7 mm
- net Net-(J15-Pin_2): track 20.6 -> 11.7 mm
- net +12V: track 318.0 -> 312.6 mm
- net Net-(J29-Pin_1): track 34.6 -> 32.8 mm

Commit message: Split
Parts:
- removed J38: 5V Lights, SMD-Connectors:SMD-PinHeader_1x04_P2.54mm_Vertical
- added C40: 100nf, Capacitor_SMD:C_1210_3225Metric, F.Cu at (32.1, 181.7)
- added C41: 100nf, Capacitor_SMD:C_1210_3225Metric, F.Cu at (81.7, 182.1)
- added C42: 100nf, Capacitor_SMD:C_1210_3225Metric, F.Cu at (130.9, 179.8)
- added J18: Conn_01x04_Pin, SMD-Connectors:SMD-PinHeader_1x04_P2.54mm_Vertical, F.Cu at (27.4, 121.9)
- added J20: 12V Lights 5 / 6, SMD-Connectors:SMD-PinHeader_1x04_P2.54mm_Vertical, F.Cu at (27.4, 72.4)
- added R30: R4K7, Resistor_SMD:R_1206_3216Metric, F.Cu at (49.1, 144.7)
- added R33: R4K7, Resistor_SMD:R_1206_3216Metric, F.Cu at (98.9, 144.7)
- added R37: R4K7, Resistor_SMD:R_1206_3216Metric, F.Cu at (150.6, 142.4)
- added U14: DS18B20, Sensor:DS18B20_SMD, F.Cu at (33.9, 174.6)
- added U15: DS18B20, Sensor:DS18B20_SMD, F.Cu at (83.5, 175.2)
- added U16: DS18B20, Sensor:DS18B20_SMD, F.Cu at (134.2, 174.3)
- J10, J9: value Conn_01x02_Pin -> Conn_01x04_Pin; footprint SMD-Connectors:SMD-PinHeader_1x02_P2.54mm_Vertical -> SMD-Connectors:SMD-PinHeader_1x04_P2.54mm_Vertical
- J15: value Conn_01x02_Pin -> 5V Lights 1 / 2; footprint SMD-Connectors:SMD-PinHeader_1x02_P2.54mm_Vertical -> SMD-Connectors:SMD-PinHeader_1x04_P2.54mm_Vertical
- J16: value Conn_01x02_Pin -> 5V Lights 3 / 4; footprint SMD-Connectors:SMD-PinHeader_1x02_P2.54mm_Vertical -> SMD-Connectors:SMD-PinHeader_1x04_P2.54mm_Vertical
- moved J15 110.8 mm to (27.4, 44.4), turned to 0 degrees
- moved C18 94.2 mm to (138.4, 47.9)
- moved C23 94.2 mm to (138.4, 74.0)
- moved C28 94.2 mm to (191.2, 79.3)
- moved R13 94.2 mm to (138.4, 43.2)
- moved R24 94.2 mm to (191.2, 83.7)
- moved C29 94.2 mm to (199.4, 45.2)
- moved C31 94.2 mm to (199.4, 79.3)
- moved J29 94.2 mm to (159.7, 37.6)
- moved R18 94.2 mm to (138.4, 78.9)
- moved R21 94.2 mm to (199.4, 41.3)
- moved R29 94.2 mm to (199.4, 83.7)
- moved SW1 94.2 mm to (144.5, 55.4)
- moved SW2 94.2 mm to (144.5, 66.5)
- moved SW3 94.2 mm to (192.8, 69.9)
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Connections:
- R10 pad 1: Net-(J15-Pin_2) -> Net-(J10-Pin_2)
- R15 pad 1: Net-(J15-Pin_1) -> Net-(J10-Pin_1)
- R2 pad 1: Net-(J16-Pin_2) -> Net-(J18-Pin_2)
- R6 pad 1: Net-(J16-Pin_1) -> Net-(J18-Pin_1)
- U3 pad 10: Net-(J17-Pin_3) -> Net-(J16-Pin_2)
- U3 pad 11: Net-(J38-Pin_4) -> Net-(J16-Pin_3)
- U3 pad 12: Net-(J17-Pin_4) -> Net-(J17-Pin_2)
- U3 pad 14: Net-(J10-Pin_1) -> Net-(J20-Pin_1)
- U3 pad 15: Net-(J17-Pin_5) -> Net-(J20-Pin_2)
- U3 pad 16: Net-(J10-Pin_2) -> Net-(J20-Pin_3)
- U3 pad 17: unconnected-(U3-GPIO13-Pad17) -> Net-(J17-Pin_3)
- U3 pad 19: /Extractor PWM -> Net-(J17-Pin_4)
- U3 pad 20: /Extractor Power -> Net-(J17-Pin_5)
- U3 pad 21: unconnected-(U3-GPIO16-Pad21) -> /Extractor PWM
- U3 pad 22: /Extractor Feedback -> unconnected-(U3-GPIO17-Pad22)
- U3 pad 32: unconnected-(U3-GPIO27_ADC1-Pad32) -> /Extractor Power
- U3 pad 34: unconnected-(U3-GPIO28_ADC2-Pad34) -> /Extractor Feedback
- U3 pad 4: Net-(J38-Pin_1) -> Net-(J15-Pin_1)
- U3 pad 5: Net-(J17-Pin_1) -> Net-(J15-Pin_2)
- U3 pad 6: Net-(J38-Pin_2) -> Net-(J15-Pin_3)
- U3 pad 7: Net-(J17-Pin_2) -> Net-(J17-Pin_1)
- U3 pad 9: Net-(J38-Pin_3) -> Net-(J16-Pin_1)
Routing:
- net +5V(B): track 128.5 -> 234.3 mm
- net +5V(C): track 132.0 -> 237.5 mm
- net Net-(J9-Pin_4): track 0.00 -> 102.6 mm
- net +3.3V: track 311.5 -> 408.8 mm
- net Net-(J10-Pin_4): track 0.00 -> 96.1 mm
- net Net-(J18-Pin_4): track 0.00 -> 96.1 mm
- net +12V: track 312.6 -> 403.2 mm
- net Net-(J9-Pin_3): track 0.00 -> 86.9 mm
- net Net-(J10-Pin_3): track 0.00 -> 83.7 mm
- net Net-(J18-Pin_3): track 0.00 -> 83.3 mm
- net /Extractor Feedback: track 96.6 -> 62.1 mm
- net /Extractor Power: track 11.5 -> 36.0 mm
- net Net-(J18-Pin_2): track 0.00 -> 18.4 mm
- net Net-(J17-Pin_3): track 37.5 -> 55.0 mm
- net Net-(J38-Pin_4): track 16.1 -> 0.00 mm
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
Commit message: Updates
Parts:
- removed C34, C38: 220uf, Capacitor_SMD:CP_Elec_8x10.5
- removed C37, C39: 100nf, Capacitor_SMD:C_1210_3225Metric
- removed D2, D3: 1N5819WS, Diode_SMD:D_SOD-323
- removed J18: Conn_01x04_Pin, SMD-Connectors:SMD-PinHeader_1x04_P2.54mm_Vertical
- removed J20: 12V Lights 5 / 6, SMD-Connectors:SMD-PinHeader_1x04_P2.54mm_Vertical
- removed J35: Extractor 2, SMD-Connectors:SMD-PinHeader_1x04_P2.54mm_Vertical
- removed J36: Extractor 3, SMD-Connectors:SMD-PinHeader_1x04_P2.54mm_Vertical
- removed Q7: PMV20XNER, ul_PMV20XNER:SOT23-TO-236AB_NEX
- removed R31: 1K, Resistor_SMD:R_1206_3216Metric_Pad1.30x1.75mm_HandSolder
- removed R32, R35: 10K, Resistor_SMD:R_1206_3216Metric_Pad1.30x1.75mm_HandSolder
- added C43: 100nf, Capacitor_SMD:C_1210_3225Metric_Pad1.33x2.70mm_HandSolder, F.Cu at (190.2, 130.8)
- added C44: 100nf, Capacitor_SMD:C_1210_3225Metric_Pad1.33x2.70mm_HandSolder, F.Cu at (183.9, 119.4)
- added C45: 220uf, Capacitor_SMD:CP_Elec_8x10.5, F.Cu at (89.0, 43.1)
- added C46: 100nf, Capacitor_SMD:C_1210_3225Metric, F.Cu at (92.5, 50.8)
- added D4: 1N5819WS, Diode_SMD:D_SOD-323, F.Cu at (92.6, 54.3)
- added J21: Sensors, SMD-Connectors:SMD-PinHeader_1x04_P2.54mm_Vertical, F.Cu at (24.1, 83.2)
- added J24: Electronics Fan, SMD-Connectors:SMD-PinHeader_1x02_P2.54mm_Vertical, F.Cu at (86.9, 54.6)
- added J25: 5V Lights 1, SMD-Connectors:SMD-PinHeader_1x04_P2.54mm_Vertical, F.Cu at (31.8, 43.9)
- added J26: 5V Lights 2, SMD-Connectors:SMD-PinHeader_1x04_P2.54mm_Vertical, F.Cu at (31.8, 51.3)
- added J28: 12V Lights, SMD-Connectors:SMD-PinHeader_1x04_P2.54mm_Vertical, F.Cu at (31.8, 59.7)
- added Q9: PMV20XNER, ul_PMV20XNER:SOT23-TO-236AB_NEX, F.Cu at (30.9, 72.0)
- added R38: 10K, Resistor_SMD:R_1206_3216Metric_Pad1.30x1.75mm_HandSolder, F.Cu at (204.0, 121.9)
- added R39: 10K, Resistor_SMD:R_1206_3216Metric_Pad1.30x1.75mm_HandSolder, F.Cu at (204.0, 124.5)
- added R43: R220, Resistor_SMD:R_1206_3216Metric, F.Cu at (32.6, 65.9)
- added R44: R10K, Resistor_SMD:R_1206_3216Metric, F.Cu at (29.2, 65.8)
- added U17: TSL2561T, TSL2561T:TMB-6_TSL2561T_AMS, F.Cu at (190.5, 125.7)
- added U18: SHT30-DIS, Sensor_Humidity:Sensirion_DFN-8-1EP_2.5x2.5mm_P0.5mm_EP1.1x1.7mm, F.Cu at (184.2, 125.7)
- C36: value 220uf -> 1000uf; footprint Capacitor_SMD:CP_Elec_8x10.5 -> Capacitor_SMD:CP_Elec_10x10.5
- J10: value Conn_01x04_Pin -> 12V Lights
- J15: value 5V Lights 1 / 2 -> 5V Lights 1
- J16: value 5V Lights 3 / 4 -> 5V Lights 2
- J9: value Conn_01x04_Pin -> I2C Sensors; footprint SMD-Connectors:SMD-PinHeader_1x04_P2.54mm_Vertical -> Connector_PinHeader_2.54mm:PinHeader_1x04_P2.54mm_Vertical; moved to B.Cu
- moved J16 80.2 mm to (76.5, 121.9), turned to 180 degrees
- moved J15 77.5 mm to (27.4, 121.9), turned to 180 degrees
- moved J9 73.3 mm to (199.4, 129.5), turned to 0 degrees
- moved J10 50.1 mm to (126.5, 121.9)
- moved R34 17.8 mm to (68.3, 87.6)
- moved Q8 17.8 mm to (73.5, 88.9)
- moved R36 17.8 mm to (68.3, 90.2)
- moved D1 15.3 mm to (90.6, 76.4), turned to 90 degrees
- moved C36 13.5 mm to (89.8, 66.0), turned to 0 degrees
- moved C35 10.6 mm to (94.8, 76.1), turned to -90 degrees
- moved J13 6.21 mm to (32.2, 31.8)
- moved J1 3.82 mm to (65.5, 27.9)
- moved J14 3.82 mm to (91.6, 27.9)
- moved J17 3.82 mm to (43.7, 26.2)
- moved U3 3.82 mm to (50.9, 61.0)
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Connections:
- C35 pad 1: Net-(D1-A) -> GND
- C36 pad 1: +12V -> GND
- C36 pad 2: Net-(D1-A) -> +12V
- C40 pad 1: Net-(J18-Pin_4) -> Net-(J15-Pin_3)
- C41 pad 1: Net-(J10-Pin_4) -> Net-(J16-Pin_3)
- C42 pad 1: Net-(J9-Pin_4) -> Net-(J10-Pin_3)
- D1 pad 2: Net-(D1-A) -> GND
- J10 pad 4: Net-(J10-Pin_4) -> GND
- J15 pad 4: +3.3V -> GND
- J16 pad 4: +3.3V -> GND
- J34 pad 2: unconnected-(J34-Pin_2-Pad2) -> /Extractor Feedback
- J34 pad 4: Net-(D1-A) -> GND
- J9 pad 1: Net-(J9-Pin_1) -> +3.3V
- J9 pad 2: Net-(J9-Pin_2) -> GND
- R10 pad 1: Net-(J10-Pin_2) -> Net-(J16-Pin_1)
- R15 pad 1: Net-(J10-Pin_1) -> Net-(J16-Pin_1)
- R2 pad 1: Net-(J18-Pin_2) -> Net-(J15-Pin_1)
- R20 pad 1: Net-(J9-Pin_2) -> Net-(J10-Pin_1)
- R26 pad 1: Net-(J9-Pin_1) -> Net-(J10-Pin_1)
- R30 pad 1: Net-(J18-Pin_3) -> Net-(J15-Pin_2)
- R30 pad 2: Net-(J18-Pin_4) -> Net-(J15-Pin_3)
- R33 pad 1: Net-(J10-Pin_3) -> Net-(J16-Pin_2)
- R33 pad 2: Net-(J10-Pin_4) -> Net-(J16-Pin_3)
- R37 pad 1: Net-(J9-Pin_3) -> Net-(J10-Pin_2)
- R37 pad 2: Net-(J9-Pin_4) -> Net-(J10-Pin_3)
- R6 pad 1: Net-(J18-Pin_1) -> Net-(J15-Pin_1)
- U14 pad 2: Net-(J18-Pin_3) -> Net-(J15-Pin_2)
- U14 pad 3: Net-(J18-Pin_4) -> Net-(J15-Pin_3)
- U15 pad 2: Net-(J10-Pin_3) -> Net-(J16-Pin_2)
- U15 pad 3: Net-(J10-Pin_4) -> Net-(J16-Pin_3)
- U16 pad 2: Net-(J9-Pin_3) -> Net-(J10-Pin_2)
- U16 pad 3: Net-(J9-Pin_4) -> Net-(J10-Pin_3)
- U3 pad 10: Net-(J16-Pin_2) -> Net-(J28-Pin_2)
- U3 pad 11: Net-(J16-Pin_3) -> /Cooling PWM
- U3 pad 12: Net-(J17-Pin_2) -> Net-(J17-Pin_1)
- U3 pad 14: Net-(J20-Pin_1) -> Net-(J17-Pin_2)
- U3 pad 15: Net-(J20-Pin_2) -> Net-(J17-Pin_3)
- U3 pad 16: Net-(J20-Pin_3) -> Net-(J17-Pin_4)
- U3 pad 17: Net-(J17-Pin_3) -> Net-(J17-Pin_5)
- U3 pad 19: Net-(J17-Pin_4) -> Net-(J21-Pin_3)
- U3 pad 20: Net-(J17-Pin_5) -> Net-(J21-Pin_4)
- U3 pad 22: unconnected-(U3-GPIO17-Pad22) -> /Extractor Feedback
- U3 pad 32: /Extractor Power -> unconnected-(U3-GPIO27_ADC1-Pad32)
- U3 pad 34: /Extractor Feedback -> unconnected-(U3-GPIO28_ADC2-Pad34)
- U3 pad 4: Net-(J15-Pin_1) -> Net-(J25-Pin_1)
- U3 pad 5: Net-(J15-Pin_2) -> Net-(J25-Pin_2)
- U3 pad 6: Net-(J15-Pin_3) -> Net-(J26-Pin_1)
- U3 pad 7: Net-(J17-Pin_1) -> Net-(J26-Pin_2)
- U3 pad 9: Net-(J16-Pin_1) -> Net-(J28-Pin_1)
Routing:
- net Net-(D1-A): track 185.6 -> 0.00 mm
- net Net-(J10-Pin_4): track 96.1 -> 0.00 mm
- net Net-(J18-Pin_4): track 96.1 -> 0.00 mm
- net Net-(J15-Pin_3): track 11.4 -> 96.2 mm
- net Net-(J16-Pin_3): track 11.9 -> 96.2 mm
- net Net-(J9-Pin_4): track 102.6 -> 18.3 mm
- net Net-(J18-Pin_3): track 83.3 -> 0.00 mm
- net Net-(D4-A): track 0.00 -> 80.4 mm, vias 0 -> 2
- net Net-(J15-Pin_2): track 11.4 -> 82.2 mm
- net Net-(J16-Pin_2): track 11.9 -> 82.6 mm
- net +3.3V: track 408.8 -> 478.7 mm
- net Net-(J9-Pin_3): track 86.9 -> 20.0 mm
- net Net-(J10-Pin_2): track 19.0 -> 85.8 mm
- net Net-(J34-Pin_1): track 77.1 -> 15.7 mm, vias 4 -> 0
- net +12V: track 403.2 -> 365.9 mm
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Other:
- board text added: "+12V IN"
- board text added: "+5V IN"
- board text added: "- | + L6"
- board text added: "1*"
- board text added: "12V PWM"
- board text added: "3.3V GND SDA SCL"
- board text added: "CTL* BTT BTB ENA ENB SW 3.3V GND"
- board text added: "DEBUG"
- board text added: "DSP* CS SC RES SDA SCL 3.3V GND"
- board text added: "GND 3.3V TMP L2 L1"
- board text added: "GND 3.3V TMP L4 L3"
- board text added: "GND 3.3V TMP L6 L5"
- board text added: "GND 3.3V TMP LGT"
- board text added: "GND| 12V| TAC| PWM"
- board text added: "L5 - | +"

Commit message: Updates
Parts:
- removed C35: 100nf, Capacitor_SMD:C_1210_3225Metric
- removed C36: 1000uf, Capacitor_SMD:CP_Elec_10x10.5
- removed C43, C44: 100nf, Capacitor_SMD:C_1210_3225Metric_Pad1.33x2.70mm_HandSolder
- removed D1: 1N5819WS, Diode_SMD:D_SOD-323
- removed Q8: A2SHB, ul_PMV20XNER:SOT23-TO-236AB_NEX
- removed R34: 1K, Resistor_SMD:R_1206_3216Metric_Pad1.30x1.75mm_HandSolder
- removed R36, R38, R39: 10K, Resistor_SMD:R_1206_3216Metric_Pad1.30x1.75mm_HandSolder
- removed U17: TSL2561T, TSL2561T:TMB-6_TSL2561T_AMS
- removed U18: SHT30-DIS, Sensor_Humidity:Sensirion_DFN-8-1EP_2.5x2.5mm_P0.5mm_EP1.1x1.7mm
- added J18: Conn_01x04_Pin, SMD-Connectors:SMD-PinHeader_1x04_P2.54mm_Vertical, F.Cu at (126.2, 86.4)
- added J20: Conn_01x04_Pin, SMD-Connectors:SMD-PinHeader_1x04_P2.54mm_Vertical, F.Cu at (144.7, 86.4)
- added R31: 1K, Resistor_SMD:R_1206_3216Metric_Pad1.30x1.75mm_HandSolder, F.Cu at (76.2, 77.5)
- moved J9 74.7 mm to (138.4, 86.4), turned to 180 degrees
- moved C31 26.2 mm to (175.6, 68.4)
- moved J29 26.2 mm to (135.8, 26.7)
- moved SW3 26.2 mm to (168.9, 59.0)
- moved SW1 26.2 mm to (120.7, 44.5)
- moved SW2 26.2 mm to (120.7, 55.6)
- moved C18 26.2 mm to (114.5, 36.9)
- moved C23 26.2 mm to (114.5, 63.1)
- moved C29 26.2 mm to (175.6, 34.3)
- moved R13 26.2 mm to (114.6, 32.2)
- moved R21 26.2 mm to (175.6, 30.4)
- moved C28 26.2 mm to (167.4, 68.4)
- moved R18 26.2 mm to (114.6, 67.9)
- moved R24 26.2 mm to (167.4, 72.7)
- moved R29 26.2 mm to (175.5, 72.7)
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Connections:
- J34 pad 1: Net-(J34-Pin_1) -> /Extractor PWM
- U3 pad 27: unconnected-(U3-GPIO21-Pad27) -> Net-(J22-Pin_6)
- U3 pad 29: Net-(J22-Pin_6) -> Net-(J22-Pin_7)
- U3 pad 31: Net-(J22-Pin_7) -> unconnected-(U3-GPIO26_ADC0-Pad31)
Routing:
- net +3.3V: track 478.7 -> 439.8 mm
- net +12V: track 365.9 -> 339.8 mm
- net /Extractor PWM: track 8.83 -> 30.5 mm
- net Net-(J34-Pin_1): track 15.7 -> 0.00 mm
- net GND: track 7.29 -> 0.00 mm
- net Net-(Q8-G): track 5.26 -> 0.00 mm
- net Net-(J22-Pin_7): track 12.9 -> 9.29 mm
- net /Extractor Feedback: track 29.7 -> 32.7 mm
- net Net-(J18-Pin_3): track 20.0 -> 18.5 mm
- net Net-(J22-Pin_6): track 10.3 -> 9.29 mm
- net Net-(J27-Pin_3): vias 0 -> 1
- net Net-(J27-Pin_1): vias 0 -> 1
- net Net-(J19-GND2): vias 0 -> 1
- net Net-(J19-GND1): vias 0 -> 1
- net Net-(J11-GND2): vias 0 -> 1
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- added copper zone on B.Cu, net Net-(J11-GND1)
- added copper zone on B.Cu, net Net-(J11-GND2)
- added copper zone on B.Cu, net Net-(J19-GND1)
- added copper zone on B.Cu, net Net-(J19-GND2)
- added copper zone on B.Cu, net Net-(J27-Pin_1)
- added copper zone on B.Cu, net Net-(J27-Pin_3)
Other:
- board text added: "+12V"
- board text added: "+5V"
- board text added: "3.3V GND SCL SDA"
- board text added: "DSP* CS DC RES SDA SCL 3.3V GND"
- board text added: "GND 3.3V TMP L"
- board text removed: "DSP* CS SC RES SDA SCL 3.3V GND"
- board text removed: "GND 3.3V TMP L2 L1"
- board text removed: "GND 3.3V TMP L4 L3"
- board text removed: "GND 3.3V TMP L6 L5"
