File: Work Bench 3.0.kicad_sch (KiCad schematic)
At the start: 136 parts, among them J1 GND(A), J10 Lights 1 GND, J11 USB_A_Stacked, J12 Lights 2 GND, J13 Conn_01x02_Pin, J14 Lights 5V+(B), J15 Lights 1 GND, J16 Lights +5V(B), J17 Controls, J18 Lights 3 GND, J19 USB_A_Stacked, J2 GND(B), J20 Lights 4 GND, J21 Lights 4 GND, J22 Display, J23 Lights +5V(c), J24 Lights +5V(C), J25 Lights 3 GND, J26 Lights 5 GND, J27 Screw_Terminal_01x04, J28 Lights 6 GND, J29 Controls, J3 GND(C), J30 Lights 6 GND, J31 Lights +12V, J32 Lights +12V, J33 Lights 5 GND, J34 Extractor 1, J35 Extractor 2, J36 Extractor 3, J4 GND(12V), J5 +5V(A), J6 +5V(B), J7 +5V(C), J8 +12V, J9 Lights 2 GND, Q1 PMV20XNEAR, Q2 PMV20XNEAR, Q3 PMV20XNEAR, Q4 PMV20XNEAR, Q5 PMV20XNEAR, Q6 PMV20XNEAR, Q7 PMV20XNER, Q8 A2SHB, SW1 FSM4JSMA, SW2 FSM4JSMA, SW3 RotaryEncoder_Switch, U1 BCP5610TA, U10 BCP5610TA, U11 BCP53TA, U12 BCP5610TA, U13 BCP53TA, U2 BCP53TA, U3 Pico, U4 BCP5610TA, U5 BCP53TA, U6 BCP5610TA, U7 BCP53TA, U8 BCP5610TA, U9 BCP53TA

Commit message: Done
Parts:
- removed J10, J15: Lights 1 GND, Connector_Wire:SolderWirePad_1x01_SMD_5x10mm, symbol Connector:Conn_01x01_Pin
- removed J16: Lights +5V(B), Connector_Wire:SolderWirePad_1x01_SMD_5x10mm, symbol Connector:Conn_01x01_Pin
- removed J18, J25: Lights 3 GND, Connector_Wire:SolderWirePad_1x01_SMD_5x10mm, symbol Connector:Conn_01x01_Pin
- removed J20, J21: Lights 4 GND, Connector_Wire:SolderWirePad_1x01_SMD_5x10mm, symbol Connector:Conn_01x01_Pin
- removed J23: Lights +5V(c), Connector_Wire:SolderWirePad_1x01_SMD_5x10mm, symbol Connector:Conn_01x01_Pin
- removed J24: Lights +5V(C), Connector_Wire:SolderWirePad_1x01_SMD_5x10mm, symbol Connector:Conn_01x01_Pin
- removed J26, J33: Lights 5 GND, Connector_Wire:SolderWirePad_1x01_SMD_5x10mm, symbol Connector:Conn_01x01_Pin
- removed J28, J30: Lights 6 GND, Connector_Wire:SolderWirePad_1x01_SMD_5x10mm, symbol Connector:Conn_01x01_Pin
- removed J31, J32: Lights +12V, Connector_Wire:SolderWirePad_1x01_SMD_5x10mm, symbol Connector:Conn_01x01_Pin
- removed J9: Lights 2 GND, Connector_Wire:SolderWirePad_1x01_SMD_5x10mm, symbol Connector:Conn_01x01_Pin
- added J10, J9: Conn_01x02_Pin, SMD-Connectors:SMD-PinHeader_1x02_P2.54mm_Vertical, symbol Connector:Conn_01x02_Pin
- added J37: Conn_01x04_Pin, SMD-Connectors:SMD-PinHeader_1x04_P2.54mm_Vertical, symbol Connector:Conn_01x04_Pin
- added J38: 5V Lights, SMD-Connectors:SMD-PinHeader_1x04_P2.54mm_Vertical, symbol Connector:Conn_01x04_Pin
- J12: value Lights 2 GND -> GND(12V)
- J14: value Lights 5V+(B) -> +12V
Connections:
- net +12V: now also C22.1, C24.1, J14.1 (Pin_1), J27.2 (Pin_2), J27.4 (Pin_4)
- net +5V(B): now also C6.1, C8.1, J11.1 (VBUS1), J11.5 (VBUS2); no longer J14.1 (Pin_1)
- net +5V(C): now also C13.1, C14.1, J19.1 (VBUS1), J19.5 (VBUS2)
- net GND: now also J12.1 (Pin_1)
- net at C22.2, J27.1 (Pin_1): now also Q6.3 (D)
- net at C24.2, J27.3 (Pin_3): now also Q5.3 (D)
- net at C13.2, J19.4 (GND1): now also Q4.3 (D)
- net at C8.2, J11.8 (GND2): now also Q1.3 (D); no longer J12.1 (Pin_1)
- net at Q3.3 (D): now also C14.2, J19.8 (GND2)
- net at C6.2, J11.4 (GND1): now also Q2.3 (D)
- net Lights 1 Signal: no longer names the net of U3.4 (GPIO2)
- net Lights 1 Signal: now also J38.1 (Pin_1); no longer R6.1
- net Lights 2 Signal: no longer names the net of R2.1
- net Lights 2 Signal: now also J37.2 (Pin_2); no longer U3.6 (GPIO4)
- net Lights 3 Signal: no longer names the net of U3.9 (GPIO6)
- net Lights 3 Signal: now also J38.3 (Pin_3); no longer R15.1
- net Lights 4 Signal: no longer names the net of R10.1
- net Lights 4 Signal: now also J37.4 (Pin_4); no longer U3.11 (GPIO8)
- net Lights 5 Signal: no longer names the net of U3.14 (GPIO10)
- net Lights 5 Signal: now also J10.1 (Pin_1); no longer R26.1
- net Lights 6 Signal: no longer names the net of R20.1
- net Lights 6 Signal: now also J9.2 (Pin_2); no longer U3.16 (GPIO12)
- new net: J38.2 (Pin_2), U3.6 (GPIO4)
- new net: J38.4 (Pin_4), U3.11 (GPIO8)
- new net: J10.2 (Pin_2), U3.16 (GPIO12)
- new net: J37.1 (Pin_1), R6.1
- new net: J37.3 (Pin_3), R15.1
- new net: J9.1 (Pin_1), R26.1
Other:
- moved on the sheet: C10, C11, C12, C13, C14, C15, C16, C17, C19, C20, C21, C22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

Commit message: Split
Parts:
- removed J37: Conn_01x04_Pin, SMD-Connectors:SMD-PinHeader_1x04_P2.54mm_Vertical, symbol Connector:Conn_01x04_Pin
- added J15, J16: Conn_01x02_Pin, SMD-Connectors:SMD-PinHeader_1x02_P2.54mm_Vertical, symbol Connector:Conn_01x02_Pin
Connections:
- net at R2.1: now also J16.2 (Pin_2)
- net at R10.1: now also J15.2 (Pin_2)
- net at R6.1: now also J16.1 (Pin_1)
- net at R15.1: now also J15.1 (Pin_1)
Changed lines of the file:
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@@
 	(wire
 		(pts
+			(xy 231.14 116.84) (xy 247.65 116.84)
+		)
+		(stroke
+			(width 0)
+			(type default)
+		)
+	)
+	(wire
+		(pts
 			(xy 77.47 313.69) (xy 77.47 318.77)
 		)
@@
 	(wire
 		(pts
-			(xy 243.84 114.3) (xy 234.95 114.3)
-		)
-		(stroke
-			(width 0)
-			(type default)
-		)
-	)
-	(wire
-		(pts
 			(xy 62.23 78.74) (xy 62.23 93.98)
 		)
@@
 	(wire
 		(pts
-			(xy 234.95 121.92) (xy 243.84 121.92)
-		)
-		(stroke
-			(width 0)
-			(type default)
-		)
-	)
-	(wire
-		(pts
 			(xy 426.72 92.71) (xy 435.61 92.71)
 		)
@@
 	(wire
 		(pts
-			(xy 234.95 119.38) (xy 247.65 119.38)
-		)
-		(stroke
-			(width 0)
-			(type default)
-		)
-	)
-	(wire
-		(pts
 			(xy 125.73 133.35) (xy 125.73 138.43)
 		)
@@
 	(wire
 		(pts
-			(xy 234.95 116.84) (xy 247.65 116.84)
-		)
-		(stroke
-			(width 0)
-			(type default)
-		)
-	)
-	(wire
-		(pts
 			(xy 377.19 86.36) (xy 403.86 86.36)
 		)
@@
 	(wire
 		(pts
+			(xy 231.14 119.38) (xy 247.65 119.38)
+		)
+		(stroke
+			(width 0)
+			(type default)
+		)
+	)
+	(wire
+		(pts
 			(xy 243.84 58.42) (xy 243.84 114.3)
 		)
@@
 	(wire
 		(pts
+			(xy 231.14 121.92) (xy 243.84 121.92)
+		)
+		(stroke
+			(width 0)
+			(type default)
+		)
+	)
+	(wire
+		(pts
 			(xy 308.61 261.62) (xy 308.61 262.89)
 		)
@@
 	(wire
 		(pts
+			(xy 231.14 114.3) (xy 243.84 114.3)
+		)
+		(stroke
+			(width 0)
+			(type default)
+		)
+	)
+	(wire
+		(pts
 			(xy 330.2 77.47) (xy 330.2 71.12)
 		)
@@
 	)
 	(symbol
+		(lib_id "Connector:Conn_01x02_Pin")
+		(at 226.06 119.38 0)
+		(unit 1)
+		(exclude_from_sim no)
+		(in_bom yes)
+		(on_board yes)
+		(dnp no)
+		(fields_autoplaced yes)
+		(property "Reference" "J15"
+			(at 226.695 114.3 0)
+			(effects
+				(font
+					(size 1.27 1.27)
+				)
+			)
+		)
+		(property "Value" "Conn_01x02_Pin"
+			(at 226.695 116.84 0)
+			(effects
+				(font
+					(size 1.27 1.27)
+				)
+			)
+		)
+		(property "Footprint" "SMD-Connectors:SMD-PinHeader_1x02_P2.54mm_Vertical"
+			(at 226.06 119.38 0)
+			(effects
+				(font
+					(size 1.27 1.27)
+				)
+				(hide yes)
+			)
+		)
+		(property "Datasheet" "~"
+			(at 226.06 119.38 0)
+			(effects
+				(font
+					(size 1.27 1.27)
+				)
+				(hide yes)
+			)
+		)
+		(property "Description" "Generic connector, single row, 01x02, script generated"
+			(at 226.06 119.38 0)
+			(effects
+				(font
+					(size 1.27 1.27)
+				)
+				(hide yes)
+			)
+		)
+		(pin "2"
+		)
+		(pin "1"
+		)
+		(instances
+			(project "Work Bench 3.0"
+				(path "/fca18d2c-2c7a-4282-a0fc-794620680e78"
+					(reference "J15")
+					(unit 1)
+				)
+			)
+		)
+	)
+	(symbol
 		(lib_id "power:GND")
 		(at 332.74 179.07 0)
@@
 	)
 	(symbol
-		(lib_id "Connector:Conn_01x04_Pin")
-		(at 229.87 116.84 0)
-		(unit 1)
-		(exclude_from_sim no)
-		(in_bom yes)
-		(on_board yes)
-		(dnp no)
-		(property "Reference" "J37"
-			(at 230.505 109.22 0)
-			(effects
-				(font
-					(size 1.27 1.27)
-				)
-			)
-		)
-		(property "Value" "Conn_01x04_Pin"
-			(at 230.505 111.76 0)
-			(effects
-				(font
-					(size 1.27 1.27)
-				)
-			)
-		)
-		(property "Footprint" "SMD-Connectors:SMD-PinHeader_1x04_P2.54mm_Vertical"
-			(at 229.87 116.84 0)
-			(effects
-				(font
-					(size 1.27 1.27)
-				)
-				(hide yes)
-			)
-		)
-		(property "Datasheet" "~"
-			(at 229.87 116.84 0)
-			(effects
-				(font
-					(size 1.27 1.27)
-				)
-				(hide yes)
-			)
-		)
-		(property "Description" "Generic connector, single row, 01x04, script generated"
-			(at 229.87 116.84 0)
-			(effects
-				(font
-					(size 1.27 1.27)
-				)
-				(hide yes)
-			)
-		)
-		(pin "3"
-		)
-		(pin "1"
-		)
-		(pin "4"
-		)
-		(pin "2"
-		)
-		(instances
-			(project "Work Bench 3.0"
-				(path "/fca18d2c-2c7a-4282-a0fc-794620680e78"
-					(reference "J37")
-					(unit 1)
-				)
-			)
-		)
-	)
-	(symbol
 		(lib_id "power:GND")
 		(at 59.69 294.64 0)
@@
 					(unit 1)
 				)
+			)
+		)
+	)
+	(symbol
+		(lib_id "Connector:Conn_01x02_Pin")
+		(at 226.06 114.3 0)
+		(unit 1)
+		(exclude_from_sim no)
+		(in_bom yes)
+		(on_board yes)
+		(dnp no)
+		(fields_autoplaced yes)
+		(property "Reference" "J16"
+			(at 226.695 109.22 0)
+			(effects
+				(font
+					(size 1.27 1.27)
+				)
+			)
+		)
+		(property "Value" "Conn_01x02_Pin"
+			(at 226.695 111.76 0)
+			(effects
+				(font
+					(size 1.27 1.27)
+				)
+			)
+		)
+		(property "Footprint" "SMD-Connectors:SMD-PinHeader_1x02_P2.54mm_Vertical"
+			(at 226.06 114.3 0)
+			(effects
+				(font
+					(size 1.27 1.27)
+				)
+				(hide yes)
+			)
+		)
+		(property "Datasheet" "~"
+			(at 226.06 114.3 0)
+			(effects
+				(font
+					(size 1.27 1.27)
+				)
+				(hide yes)
+			)
+		)
+		(property "Description" "Generic connector, single row, 01x02, script generated"
+			(at 226.06 114.3 0)
+			(effects
+				(font
+					(size 1.27 1.27)
+				)
+				(hide yes)
+			)
+		)
+		(pin "2"
+		)
+		(pin "1"
+		)
+		(instances
+			(project "Work Bench 3.0"
+				(path "/fca18d2c-2c7a-4282-a0fc-794620680e78"
+					(reference "J16")
+					(unit 1)
+				)

Commit message: Split
Parts:
- removed J10, J15, J16, J9: Conn_01x02_Pin, SMD-Connectors:SMD-PinHeader_1x02_P2.54mm_Vertical, symbol Connector:Conn_01x02_Pin
- removed J38: 5V Lights, SMD-Connectors:SMD-PinHeader_1x04_P2.54mm_Vertical, symbol Connector:Conn_01x04_Pin
- added C40, C41, C42: 100nf, Capacitor_SMD:C_1210_3225Metric, symbol Device:C_Small
- added J10, J18, J9: Conn_01x04_Pin, SMD-Connectors:SMD-PinHeader_1x04_P2.54mm_Vertical, symbol Connector:Conn_01x04_Pin
- added J15: 5V Lights 1 / 2, SMD-Connectors:SMD-PinHeader_1x04_P2.54mm_Vertical, symbol Connector:Conn_01x04_Pin
- added J16: 5V Lights 3 / 4, SMD-Connectors:SMD-PinHeader_1x04_P2.54mm_Vertical, symbol Connector:Conn_01x04_Pin
- added J20: 12V Lights 5 / 6, SMD-Connectors:SMD-PinHeader_1x04_P2.54mm_Vertical, symbol Connector:Conn_01x04_Pin
- added R30, R33, R37: R4K7, Resistor_SMD:R_1206_3216Metric, symbol Device:R
- added U14, U15, U16: DS18B20, Sensor:DS18B20_SMD, symbol Sensor_Temperature:DS18B20
Connections:
- net +3.3V: now also J15.4 (Pin_4), J16.4 (Pin_4), J20.4 (Pin_4)
- net Extractor Feedback: now also U3.34 (GPIO28_ADC2); no longer U3.22 (GPIO17)
- net Extractor PWM: now also U3.21 (GPIO16); no longer U3.19 (GPIO14)
- net Extractor Power: now also U3.32 (GPIO27_ADC1); no longer U3.20 (GPIO15)
- net GND: now also C40.2, C41.2, C42.2, U14.1 (GND), U15.1 (GND), U16.1 (GND)
- net at R20.1: now also J9.2 (Pin_2)
- net at R2.1: now also J18.2 (Pin_2)
- net at R10.1: now also J10.2 (Pin_2)
- net at U3.4 (GPIO2): now also J15.1 (Pin_1)
- net at U3.6 (GPIO4): now also J15.3 (Pin_3)
- net at U3.9 (GPIO6): now also J16.1 (Pin_1)
- net at U3.11 (GPIO8): now also J16.3 (Pin_3)
- net at U3.10 (GPIO7): now also J16.2 (Pin_2); no longer J17.3 (Pin_3)
- net at U3.12 (GPIO9): now also J17.2 (Pin_2); no longer J17.4 (Pin_4)
- net at U3.14 (GPIO10): now also J20.1 (Pin_1)
- net at U3.15 (GPIO11): now also J20.2 (Pin_2); no longer J17.5 (Pin_5)
- net at U3.16 (GPIO12): now also J20.3 (Pin_3)
- net at U3.17 (GPIO13): now also J17.3 (Pin_3)
- net at U3.5 (GPIO3): now also J15.2 (Pin_2); no longer J17.1 (Pin_1)
- net at U3.7 (GPIO5): now also J17.1 (Pin_1); no longer J17.2 (Pin_2)
- net at R6.1: now also J18.1 (Pin_1)
- net at R15.1: now also J10.1 (Pin_1)
- net at R26.1: now also J9.1 (Pin_1)
- new net: J10.3 (Pin_3), R33.1, U15.2 (DQ)
- new net: C41.1, J10.4 (Pin_4), R33.2, U15.3 (V_{DD})
- new net: C40.1, J18.4 (Pin_4), R30.2, U14.3 (V_{DD})
- new net: J18.3 (Pin_3), R30.1, U14.2 (DQ)
- new net: J17.4 (Pin_4), U3.19 (GPIO14)
- new net: J17.5 (Pin_5), U3.20 (GPIO15)
- new net: C42.1, J9.4 (Pin_4), R37.2, U16.3 (V_{DD})
- new net: J9.3 (Pin_3), R37.1, U16.2 (DQ)
Other:
- moved on the sheet: C1, C10, C11, C12, C13, C14, C15, C16, C17, C18, C19, C2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

Commit message: Updates
Parts:
- removed C34, C38: 220uf, Capacitor_SMD:CP_Elec_8x10.5, symbol Device:C_Polarized
- removed C37, C39: 100nf, Capacitor_SMD:C_1210_3225Metric, symbol Device:C_Small
- removed D2, D3: 1N5819WS, Diode_SMD:D_SOD-323, symbol Diode:1N5819WS
- removed J18: Conn_01x04_Pin, SMD-Connectors:SMD-PinHeader_1x04_P2.54mm_Vertical, symbol Connector:Conn_01x04_Pin
- removed J20: 12V Lights 5 / 6, SMD-Connectors:SMD-PinHeader_1x04_P2.54mm_Vertical, symbol Connector:Conn_01x04_Pin
- removed J35: Extractor 2, SMD-Connectors:SMD-PinHeader_1x04_P2.54mm_Vertical, symbol Connector:Conn_01x04_Pin
- removed J36: Extractor 3, SMD-Connectors:SMD-PinHeader_1x04_P2.54mm_Vertical, symbol Connector:Conn_01x04_Pin
- removed Q7: PMV20XNER, SOT23-TO-236AB_NEX, symbol ul_PMV20XNER:PMV20XNER
- removed R31: 1K, Resistor_SMD:R_1206_3216Metric_Pad1.30x1.75mm_HandSolder, symbol Device:R
- removed R32, R35: 10K, Resistor_SMD:R_1206_3216Metric_Pad1.30x1.75mm_HandSolder, symbol Device:R
- added C43, C44: 100nf, Capacitor_SMD:C_1210_3225Metric_Pad1.33x2.70mm_HandSolder, symbol Device:C
- added C45: 220uf, Capacitor_SMD:CP_Elec_8x10.5, symbol Device:C_Polarized
- added C46: 100nf, Capacitor_SMD:C_1210_3225Metric, symbol Device:C_Small
- added D4: 1N5819WS, Diode_SMD:D_SOD-323, symbol Diode:1N5819WS
- added J21: Sensors, SMD-Connectors:SMD-PinHeader_1x04_P2.54mm_Vertical, symbol Connector:Conn_01x04_Pin
- added J24: Electronics Fan, SMD-Connectors:SMD-PinHeader_1x02_P2.54mm_Vertical, symbol Connector:Conn_01x02_Pin
- added J25: 5V Lights 1, SMD-Connectors:SMD-PinHeader_1x04_P2.54mm_Vertical, symbol Connector:Conn_01x04_Pin
- added J26: 5V Lights 2, SMD-Connectors:SMD-PinHeader_1x04_P2.54mm_Vertical, symbol Connector:Conn_01x04_Pin
- added J28: 12V Lights, SMD-Connectors:SMD-PinHeader_1x04_P2.54mm_Vertical, symbol Connector:Conn_01x04_Pin
- added Q9: PMV20XNER, ul_PMV20XNER:SOT23-TO-236AB_NEX, symbol ul_PMV20XNER:PMV20XNER
- added R38, R39: 10K, Resistor_SMD:R_1206_3216Metric_Pad1.30x1.75mm_HandSolder, symbol Device:R
- added R43: R220, Resistor_SMD:R_1206_3216Metric, symbol Device:R
- added R44: R10K, Resistor_SMD:R_1206_3216Metric, symbol Device:R
- added U17: TSL2561T, TMB-6_TSL2561T_AMS, symbol TSL2561T:TSL2561T
- added U18: SHT30-DIS, Sensor_Humidity:Sensirion_DFN-8-1EP_2.5x2.5mm_P0.5mm_EP1.1x1.7mm, symbol Sensor_Humidity:SHT30-DIS
- C36: value 220uf -> 1000uf; footprint Capacitor_SMD:CP_Elec_8x10.5 -> Capacitor_SMD:CP_Elec_10x10.5
- J10: value Conn_01x04_Pin -> 12V Lights
- J15: value 5V Lights 1 / 2 -> 5V Lights 1
- J16: value 5V Lights 3 / 4 -> 5V Lights 2
- J9: value Conn_01x04_Pin -> I2C Sensors; footprint SMD-Connectors:SMD-PinHeader_1x04_P2.54mm_Vertical -> Connector_PinHeader_2.54mm:PinHeader_1x04_P2.54mm_Vertical
Connections:
- net +12V: now also C36.2, C45.1, C46.2, D4.1 (K), J24.1 (Pin_1); no longer C36.1
- net +3.3V: now also J9.1 (Pin_1), C43.2, C44.1, J21.1 (Pin_1), J25.3 (Pin_3), J26.3 (Pin_3), J28.3 (Pin_3), R38.1, R39.1, U17.1 (VDD), U18.5 (VDD); no longer J15.4 (Pin_4), J16.4 (Pin_4)
- net Extractor Feedback: now also J34.2 (Pin_2), U3.22 (GPIO17); no longer U3.34 (GPIO28_ADC2)
- net GND: now also C35.1, C36.1, D1.2 (A), J10.4 (Pin_4), J15.4 (Pin_4), J16.4 (Pin_4), J34.4 (Pin_4), J9.2 (Pin_2), C43.1, C44.2, C45.2, J21.2 (Pin_2), J25.4 (Pin_4), J26.4 (Pin_4), J28.4 (Pin_4), Q9.2 (S), R44.1, U17.2 (ADDR_SEL), U17.3 (GND), U18.2 (ADDR), U18.7 (R), U18.8 (VSS), U18.9 (VSS)
- net at J10.1 (Pin_1): now also R20.1, R26.1; no longer R15.1
- net at R10.1: now also J16.1 (Pin_1), R15.1; no longer J10.2 (Pin_2)
- net at R33.1, U15.2 (DQ): now also J16.2 (Pin_2); no longer J10.3 (Pin_3)
- net at C41.1, R33.2, U15.3 (V_{DD}): now also J16.3 (Pin_3); no longer J10.4 (Pin_4)
- net at R2.1: now also J15.1 (Pin_1), R6.1
- net at C40.1, R30.2, U14.3 (V_{DD}): now also J15.3 (Pin_3)
- net at R30.1, U14.2 (DQ): now also J15.2 (Pin_2)
- net at U3.14 (GPIO10): now also J17.2 (Pin_2)
- net at U3.15 (GPIO11): now also J17.3 (Pin_3)
- net at U3.16 (GPIO12): now also J17.4 (Pin_4)
- net at U3.10 (GPIO7): now also J28.2 (Pin_2); no longer J16.2 (Pin_2)
- net Cooling PWM: now reaches U3.11 (GPIO8)
- net Cooling PWM: now also R43.1; no longer J16.3 (Pin_3)
- net at U3.12 (GPIO9): now also J17.1 (Pin_1); no longer J17.2 (Pin_2)
- net at U3.17 (GPIO13): now also J17.5 (Pin_5); no longer J17.3 (Pin_3)
- net at U3.19 (GPIO14): now also J21.3 (Pin_3); no longer J17.4 (Pin_4)
- net at U3.20 (GPIO15): now also J21.4 (Pin_4); no longer J17.5 (Pin_5)
- net at U3.4 (GPIO2): now also J25.1 (Pin_1); no longer J15.1 (Pin_1)
- net at U3.5 (GPIO3): now also J25.2 (Pin_2); no longer J15.2 (Pin_2)
- net at U3.6 (GPIO4): now also J26.1 (Pin_1); no longer J15.3 (Pin_3)
- net at U3.7 (GPIO5): now also J26.2 (Pin_2); no longer J17.1 (Pin_1)
- net at U3.9 (GPIO6): now also J28.1 (Pin_1); no longer J16.1 (Pin_1)
- net at C42.1, R37.2, U16.3 (V_{DD}): now also J10.3 (Pin_3); no longer J9.4 (Pin_4)
- net at R37.1, U16.2 (DQ): now also J10.2 (Pin_2); no longer J9.3 (Pin_3)
- net Extractor Power: no longer names the net of U3.32 (GPIO27_ADC1)
- new net: J9.3 (Pin_3), R39.2, U17.6 (SDA), U18.1 (SDA)
- new net: C46.1, D4.2 (A), J24.2 (Pin_2), Q9.3 (D)
- new net: Q9.1 (G), R43.2, R44.2
- new net: J9.4 (Pin_4), R38.2, U17.4 (SCL), U18.4 (SCL)
Other:
- moved on the sheet: J17

Commit message: Updates
Parts:
- removed C35: 100nf, Capacitor_SMD:C_1210_3225Metric, symbol Device:C_Small
- removed C36: 1000uf, Capacitor_SMD:CP_Elec_10x10.5, symbol Device:C_Polarized
- removed C43, C44: 100nf, Capacitor_SMD:C_1210_3225Metric_Pad1.33x2.70mm_HandSolder, symbol Device:C
- removed D1: 1N5819WS, Diode_SMD:D_SOD-323, symbol Diode:1N5819WS
- removed Q8: A2SHB, SOT23-TO-236AB_NEX, symbol ul_PMV20XNER:PMV20XNER
- removed R34: 1K, Resistor_SMD:R_1206_3216Metric_Pad1.30x1.75mm_HandSolder, symbol Device:R
- removed R36, R38, R39: 10K, Resistor_SMD:R_1206_3216Metric_Pad1.30x1.75mm_HandSolder, symbol Device:R
- removed U17: TSL2561T, TMB-6_TSL2561T_AMS, symbol TSL2561T:TSL2561T
- removed U18: SHT30-DIS, Sensor_Humidity:Sensirion_DFN-8-1EP_2.5x2.5mm_P0.5mm_EP1.1x1.7mm, symbol Sensor_Humidity:SHT30-DIS
- added J18, J20: Conn_01x04_Pin, SMD-Connectors:SMD-PinHeader_1x04_P2.54mm_Vertical, symbol Connector:Conn_01x04_Pin
- added R31: 1K, Resistor_SMD:R_1206_3216Metric_Pad1.30x1.75mm_HandSolder, symbol Device:R
Connections:
- net +3.3V: now also J18.1 (Pin_1), J20.1 (Pin_1), R31.2
- net Extractor Feedback: now also R31.1
- net Extractor PWM: now also J34.1 (Pin_1)
- net GND: now also J18.2 (Pin_2), J20.2 (Pin_2)
- net at J9.3 (Pin_3): now also J18.3 (Pin_3), J20.3 (Pin_3)
- net at U3.27 (GPIO21): now also J22.6 (Pin_6)
- net at U3.29 (GPIO22): now also J22.7 (Pin_7); no longer J22.6 (Pin_6)
- net at U3.31 (GPIO26_ADC0): no longer J22.7 (Pin_7)
- net at J9.4 (Pin_4): now also J18.4 (Pin_4), J20.4 (Pin_4)
Other:
- moved on the sheet: C1, C10, C13, C14, C17, C19, C2, C22, C24, C27, C3, C30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
